File: SensorHub/SensorHub.kicad_pcb (KiCad board)
At the start: 2 copper layers, 54 x 40 mm, 35 parts, among them J1 CS1, J2 CS2, U1 CY8C4046LQI-T452

Commit message: Images
Parts:
- removed G***: LOGO, LOGO
